File: focControllerV1/focControllerV1.kicad_sch (KiCad schematic)
At the start: 95 parts, among them J1 Conn_01x05, J2 Conn_01x05, J3 USB_C_Receptacle_USB2.0, Q1 BC818W, Q2 BC818W, SW1 SW_Push, U1 LP2992IM5X-5.0/NOPB, U10 DRV8313PWP, U11 INA240A2PW, U12 INA240A2PW, U13 INA240A2PW, U14 KF301-5.0-2P, U15 ESP32-WROOM-32, U2 ME3116AM6G, U3 DRV8313PWP, U4 INA240A2PW, U5 MPU-6050, U7 CH340C, U8 KF301-5.0-3P, U9 KF301-5.0-3P

Commit message: 728
Parts:
- C20, C34, C35, R26, R27: footprint (none) -> Capacitor_SMD:C_0603_1608Metric_Pad1.08x0.95mm_HandSolder
Connections:
- net I2C1_SCL: now also U15.30 (IO18)
- net I2C1_SDA: now also U15.31 (IO19)
- net I2C2_SCL: now also U15.33 (IO21)
- net I2C2_SDA: now also U15.36 (IO22)
- net LED: now also R12.1
Changed lines of the file:
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@@
     (effects (font (size 1.27 1.27) bold) (justify left bottom))
   )
-  (label "I2C2_SDA" (at 119.38 172.72 180) (fields_autoplaced)
-    (effects (font (size 1.27 1.27)) (justify right bottom))
+  (label "I2C2_SDA" (at 110.49 172.72 0) (fields_autoplaced)
+    (effects (font (size 1.27 1.27)) (justify left bottom))
   )
   (label "RXD" (at 320.04 49.53 0) (fields_autoplaced)
@@
     (effects (font (size 1.27 1.27)) (justify left bottom))
   )
-  (label "I2C1_SDA" (at 119.38 167.64 180) (fields_autoplaced)
-    (effects (font (size 1.27 1.27)) (justify right bottom))
+  (label "I2C1_SDA" (at 110.49 167.64 0) (fields_autoplaced)
+    (effects (font (size 1.27 1.27)) (justify left bottom))
   )
   (label "M2_OUT1_P" (at 182.88 254 180) (fields_autoplaced)
@@
     (effects (font (size 1.27 1.27) bold) (justify right bottom))
   )
+  (label "LED" (at 99.06 255.27 270) (fields_autoplaced)
+    (effects (font (size 1.27 1.27)) (justify right bottom))
+  )
   (label "M1_IN3" (at 110.49 177.8 0) (fields_autoplaced)
     (effects (font (size 1.27 1.27) bold) (justify left bottom))
@@
     (effects (font (size 1.27 1.27) bold) (justify left bottom))
   )
-  (label "I2C1_SCL" (at 119.38 165.1 180) (fields_autoplaced)
-    (effects (font (size 1.27 1.27)) (justify right bottom))
+  (label "I2C1_SCL" (at 110.49 165.1 0) (fields_autoplaced)
+    (effects (font (size 1.27 1.27)) (justify left bottom))
   )
   (label "M2_OUT3" (at 345.44 172.72 0) (fields_autoplaced)
@@
     (effects (font (size 1.27 1.27) bold) (justify left bottom))
   )
-  (label "I2C2_SCL" (at 119.38 170.18 180) (fields_autoplaced)
-    (effects (font (size 1.27 1.27)) (justify right bottom))
+  (label "I2C2_SCL" (at 110.49 170.18 0) (fields_autoplaced)
+    (effects (font (size 1.27 1.27)) (justify left bottom))
   )
   (label "EN" (at 80.01 134.62 180) (fields_autoplaced)
@@
       (effects (font (size 1.27 1.27)))
     )
-    (property "Footprint" "" (at 218.44 151.4348 0)
+    (property "Footprint" "Capacitor_SMD:C_0603_1608Metric_Pad1.08x0.95mm_HandSolder" (at 218.44 151.4348 0)
       (effects (font (size 1.27 1.27)) hide)
     )
@@
       (effects (font (size 1.27 1.27)))
     )
-    (property "Footprint" "" (at 172.72 138.938 90)
+    (property "Footprint" "Capacitor_SMD:C_0603_1608Metric_Pad1.08x0.95mm_HandSolder" (at 172.72 138.938 90)
       (effects (font (size 1.27 1.27)) hide)
     )
@@
       (effects (font (size 1.27 1.27)))
     )
-    (property "Footprint" "" (at 218.44 148.2852 0)
+    (property "Footprint" "Capacitor_SMD:C_0603_1608Metric_Pad1.08x0.95mm_HandSolder" (at 218.44 148.2852 0)
       (effects (font (size 1.27 1.27)) hide)
     )
@@
       (effects (font (size 1.27 1.27)))
     )
-    (property "Footprint" "" (at 191.77 119.6848 0)
+    (property "Footprint" "Capacitor_SMD:C_0603_1608Metric_Pad1.08x0.95mm_HandSolder" (at 191.77 119.6848 0)
       (effects (font (size 1.27 1.27)) hide)
     )
@@
       (effects (font (size 1.27 1.27)))
     )
-    (property "Footprint" "" (at 172.72 136.398 90)
+    (property "Footprint" "Capacitor_SMD:C_0603_1608Metric_Pad1.08x0.95mm_HandSolder" (at 172.72 136.398 90)
       (effects (font (size 1.27 1.27)) hide)
     )

Commit message: 729
Connections:
- net DRV1_FAULT: now also U15.22 (SDI/SD1); no longer U15.28 (IO17)
- net DRV2_FAULT: now also U15.10 (IO25); no longer U15.37 (IO23)
- net I2C1_SCL: now also U15.33 (IO21); no longer U15.30 (IO18)
- net I2C1_SDA: now also U15.36 (IO22); no longer U15.31 (IO19)
- net I2C2_SCL: now also U15.30 (IO18); no longer U15.33 (IO21)
- net I2C2_SDA: now also U15.31 (IO19); no longer U15.36 (IO22)
- net LED: now also U15.9 (IO33); no longer U15.27 (IO16)
- net M1_IN1: now also U15.27 (IO16); no longer U15.8 (IO32)
- net M1_IN2: no longer U15.9 (IO33)
- net M1_IN3: no longer U15.10 (IO25)
- net M1_OUT1_CS: now also U15.26 (IO4); no longer U15.5 (SENSOR_VN)
- net M1_OUT2_CS: now also U15.24 (IO2); no longer U15.4 (SENSOR_VP)
- net M2_OUT1_CS: now also U15.8 (IO32); no longer U15.6 (IO34)
- net M2_OUT2_CS: now also U15.16 (IO13); no longer U15.7 (IO35)
Changed lines of the file:
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@@
     (effects (font (size 2 2) (thickness 0.4) bold) (justify left bottom))
-  )
-  (label "M1_IN2" (at 110.49 187.96 0) (fields_autoplaced)
-    (effects (font (size 1.27 1.27) bold) (justify left bottom))
-  )
-  (label "I2C2_SDA" (at 110.49 172.72 0) (fields_autoplaced)
-    (effects (font (size 1.27 1.27)) (justify left bottom))
   )
   (label "RXD" (at 320.04 49.53 0) (fields_autoplaced)
     (effects (font (size 1.27 1.27)) (justify left bottom))
   )
-  (label "M2_OUT1_CS" (at 110.49 190.5 0) (fields_autoplaced)
+  (label "I2C2_SDA" (at 110.49 167.64 0) (fields_autoplaced)
     (effects (font (size 1.27 1.27)) (justify left bottom))
   )
@@
   )
   (label "D+" (at 261.62 55.88 0) (fields_autoplaced)
-    (effects (font (size 1.27 1.27)) (justify left bottom))
-  )
-  (label "I2C1_SDA" (at 110.49 167.64 0) (fields_autoplaced)
     (effects (font (size 1.27 1.27)) (justify left bottom))
   )
@@
     (effects (font (size 1.27 1.27) bold) (justify left bottom))
   )
-  (label "M1_OUT2_P" (at 323.85 133.35 180) (fields_autoplaced)
+  (label "DRV1_FAULT" (at 80.01 167.64 180) (fields_autoplaced)
     (effects (font (size 1.27 1.27) bold) (justify right bottom))
   )
-  (label "M1_OUT2_CS" (at 80.01 139.7 180) (fields_autoplaced)
+  (label "I2C1_SDA" (at 110.49 172.72 0) (fields_autoplaced)
+    (effects (font (size 1.27 1.27)) (justify left bottom))
+  )
+  (label "M1_OUT2_P" (at 323.85 133.35 180) (fields_autoplaced)
     (effects (font (size 1.27 1.27) bold) (justify right bottom))
   )
@@
     (effects (font (size 1.27 1.27)) (justify right bottom))
   )
-  (label "DRV1_FAULT" (at 110.49 162.56 0) (fields_autoplaced)
+  (label "M1_OUT1_CS" (at 110.49 144.78 0) (fields_autoplaced)
     (effects (font (size 1.27 1.27) bold) (justify left bottom))
+  )
+  (label "I2C1_SCL" (at 110.49 170.18 0) (fields_autoplaced)
+    (effects (font (size 1.27 1.27)) (justify left bottom))
   )
   (label "M1_OUT2_N" (at 242.57 217.17 180) (fields_autoplaced)
     (effects (font (size 1.27 1.27) bold) (justify right bottom))
+  )
+  (label "I2C2_SCL" (at 110.49 165.1 0) (fields_autoplaced)
+    (effects (font (size 1.27 1.27)) (justify left bottom))
+  )
+  (label "M2_OUT2_CS" (at 110.49 152.4 0) (fields_autoplaced)
+    (effects (font (size 1.27 1.27) bold) (justify left bottom))
   )
   (label "DRV1_EN" (at 110.49 157.48 0) (fields_autoplaced)
@@
     (effects (font (size 1.27 1.27) bold) (justify left bottom))
   )
-  (label "M1_OUT1_CS" (at 80.01 142.24 180) (fields_autoplaced)
-    (effects (font (size 1.27 1.27) bold) (justify right bottom))
+  (label "DRV2_FAULT" (at 110.49 177.8 0) (fields_autoplaced)
+    (effects (font (size 1.27 1.27) bold) (justify left bottom))
   )
   (label "LED" (at 99.06 255.27 270) (fields_autoplaced)
     (effects (font (size 1.27 1.27)) (justify right bottom))
-  )
-  (label "M1_IN3" (at 110.49 177.8 0) (fields_autoplaced)
-    (effects (font (size 1.27 1.27) bold) (justify left bottom))
   )
   (label "TXD" (at 110.49 137.16 0) (fields_autoplaced)
@@
     (effects (font (size 1.27 1.27) bold) (justify left bottom))
   )
-  (label "I2C1_SCL" (at 110.49 165.1 0) (fields_autoplaced)
-    (effects (font (size 1.27 1.27)) (justify left bottom))
-  )
   (label "M2_OUT3" (at 345.44 172.72 0) (fields_autoplaced)
     (effects (font (size 1.27 1.27) bold) (justify left bottom))
-  )
-  (label "LED" (at 110.49 160.02 0) (fields_autoplaced)
-    (effects (font (size 1.27 1.27)) (justify left bottom))
   )
   (label "I2C2_SCL" (at 49.53 246.38 180) (fields_autoplaced)
@@
     (effects (font (size 1.27 1.27) bold) (justify right bottom))
   )
+  (label "M2_OUT1_CS" (at 110.49 185.42 0) (fields_autoplaced)
+    (effects (font (size 1.27 1.27)) (justify left bottom))
+  )
   (label "RTS" (at 351.79 50.8 0) (fields_autoplaced)
     (effects (font (size 1.27 1.27)) (justify left bottom))
+  )
+  (label "M1_IN1" (at 110.49 160.02 0) (fields_autoplaced)
+    (effects (font (size 1.27 1.27) bold) (justify left bottom))
   )
   (label "M2_IN3" (at 110.49 154.94 0) (fields_autoplaced)
@@
     (effects (font (size 1.27 1.27)) (justify left bottom))
   )
-  (label "M2_OUT2_CS" (at 110.49 193.04 0) (fields_autoplaced)
-    (effects (font (size 1.27 1.27) bold) (justify left bottom))
-  )
   (label "I2C2_SDA" (at 49.53 254 180) (fields_autoplaced)
     (effects (font (size 1.27 1.27)) (justify right bottom))
   )
-  (label "DRV2_FAULT" (at 110.49 175.26 0) (fields_autoplaced)
-    (effects (font (size 1.27 1.27) bold) (justify left bottom))
+  (label "LED" (at 110.49 187.96 0) (fields_autoplaced)
+    (effects (font (size 1.27 1.27)) (justify left bottom))
   )
   (label "I2C1_SCL" (at 168.91 134.62 180) (fields_autoplaced)
@@
   )
   (label "M2_OUT2_CS" (at 254 259.08 0) (fields_autoplaced)
+    (effects (font (size 1.27 1.27) bold) (justify left bottom))
+  )
+  (label "M1_OUT2_CS" (at 110.49 139.7 0) (fields_autoplaced)
     (effects (font (size 1.27 1.27) bold) (justify left bottom))
   )
@@
     (effects (font (size 1.27 1.27) bold) (justify left bottom))
   )
+  (label "M1_IN3" (at 134.62 144.78 0) (fields_autoplaced)
+    (effects (font (size 1.27 1.27) bold) (justify left bottom))
+  )
   (label "M1_OUT1_N" (at 313.69 167.64 0) (fields_autoplaced)
     (effects (font (size 1.27 1.27) bold) (justify left bottom))
-  )
-  (label "M1_IN1" (at 110.49 185.42 0) (fields_autoplaced)
-    (effects (font (size 1.27 1.27) bold) (justify left bottom))
-  )
-  (label "I2C2_SCL" (at 110.49 170.18 0) (fields_autoplaced)
-    (effects (font (size 1.27 1.27)) (justify left bottom))
   )
   (label "EN" (at 80.01 134.62 180) (fields_autoplaced)
     (effects (font (size 1.27 1.27) bold) (justify right bottom))
   )
+  (label "M1_IN2" (at 132.2269 148.2068 0) (fields_autoplaced)
+    (effects (font (size 1.27 1.27) bold) (justify left bottom))
+  )
   (label "D-" (at 261.62 50.8 0) (fields_autoplaced)
