File: focControllerV1/_autosave-focControllerV1.kicad_sch (KiCad schematic)
At the start: 95 parts, among them J1 Conn_01x05, J2 Conn_01x05, J3 USB_C_Receptacle_USB2.0, Q1 BC818W, Q2 BC818W, SW1 SW_Push, U1 LP2992IM5X-5.0/NOPB, U10 DRV8313PWP, U11 INA240A2PW, U12 INA240A2PW, U13 INA240A2PW, U14 KF301-5.0-2P, U15 ESP32-WROOM-32, U2 ME3116AM6G, U3 DRV8313PWP, U4 INA240A2PW, U5 MPU-6050, U7 CH340C, U8 KF301-5.0-3P, U9 KF301-5.0-3P

Commit message: 准备布线
Parts:
- C20, C34, C35, R26, R27: footprint (none) -> Capacitor_SMD:C_0603_1608Metric_Pad1.08x0.95mm_HandSolder
Changed lines of the file:
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@@
       (effects (font (size 1.27 1.27)))
     )
-    (property "Footprint" "" (at 218.44 151.4348 0)
+    (property "Footprint" "Capacitor_SMD:C_0603_1608Metric_Pad1.08x0.95mm_HandSolder" (at 218.44 151.4348 0)
       (effects (font (size 1.27 1.27)) hide)
     )
@@
       (effects (font (size 1.27 1.27)))
     )
-    (property "Footprint" "" (at 172.72 138.938 90)
+    (property "Footprint" "Capacitor_SMD:C_0603_1608Metric_Pad1.08x0.95mm_HandSolder" (at 172.72 138.938 90)
       (effects (font (size 1.27 1.27)) hide)
     )
@@
       (effects (font (size 1.27 1.27)))
     )
-    (property "Footprint" "" (at 218.44 148.2852 0)
+    (property "Footprint" "Capacitor_SMD:C_0603_1608Metric_Pad1.08x0.95mm_HandSolder" (at 218.44 148.2852 0)
       (effects (font (size 1.27 1.27)) hide)
     )
@@
       (effects (font (size 1.27 1.27)))
     )
-    (property "Footprint" "" (at 191.77 119.6848 0)
+    (property "Footprint" "Capacitor_SMD:C_0603_1608Metric_Pad1.08x0.95mm_HandSolder" (at 191.77 119.6848 0)
       (effects (font (size 1.27 1.27)) hide)
     )
@@
       (effects (font (size 1.27 1.27)))
     )
-    (property "Footprint" "" (at 172.72 136.398 90)
-      (effects (font (size 1.27 1.27)) hide)
-    )
+    (property "Footprint" "Capacitor_SMD:C_0603_1608Metric_Pad1.08x0.95mm_HandSolder" (at 172.72 136.398 90)
+      (effects (font (size 1.27 1.27)) hide)
+    )
