File: focControllerV1/focControllerV1.kicad_pcb (KiCad board)
At the start: 2 copper layers, 86.8 x 49 mm, 95 parts, among them J1 Conn_01x05, J2 Conn_01x05, J3 USB_C_Receptacle_USB2.0, Q1 BC818W, Q2 BC818W, SW1 SW_Push, U1 LP2992IM5X-5.0/NOPB, U10 DRV8313PWP, U11 INA240A2PW, U12 INA240A2PW, U13 INA240A2PW, U14 KF301-5.0-2P, U15 ESP32-WROOM-32, U2 ME3116AM6G, U3 DRV8313PWP, U4 INA240A2PW, U5 MPU-6050, U7 CH340C, U8 KF301-5.0-3P, U9 KF301-5.0-3P

Commit message: 728
Parts:
- R8, R9: moved to F.Cu
- moved R9 38.8 mm to (62.7, 71.2), turned to 0 degrees
- moved R8 38.8 mm to (62.7, 69.1), turned to 0 degrees
- moved SW1 35.8 mm to (110.4, 76.6)
- moved C32 32.7 mm to (101.8, 69.3), turned to -90 degrees
- moved C31 30.7 mm to (99.8, 69.2), turned to -90 degrees
- moved R14 29.2 mm to (76.1, 69.5)
- moved R13 28.2 mm to (76.0, 74.5)
- moved C30 9.42 mm to (106.3, 76.2)
- moved R12 3.73 mm to (105.4, 81.2), turned to 0 degrees
- moved U7 3.50 mm to (90.4, 94.4)
- moved R11 3.18 mm to (104.0, 76.3), turned to -90 degrees
- moved C15 2.89 mm to (92.1, 99.1)
- moved R6 2.77 mm to (76.1, 71.1), turned to 0 degrees
- moved C35 2.75 mm to (49.4, 79.8)
- moved U5 2.75 mm to (53.3, 78.6)
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Connections:
- R12 pad 1: unconnected-(R12-Pad1) -> /LED
- U15 pad 30: unconnected-(U15-IO18-Pad30) -> /I2C1_SCL
- U15 pad 31: unconnected-(U15-IO19-Pad31) -> /I2C1_SDA
- U15 pad 33: unconnected-(U15-IO21-Pad33) -> /I2C2_SCL
- U15 pad 36: unconnected-(U15-IO22-Pad36) -> /I2C2_SDA
Routing:
- net +3V3: track 0.00 -> 164.1 mm, vias 0 -> 6
- net VCC: track 0.00 -> 106.5 mm, vias 0 -> 4
- net +5V: track 0.00 -> 51.6 mm, vias 0 -> 1
- net /EN: track 0.00 -> 43.6 mm, vias 0 -> 1
- net Net-(D9-A): track 0.00 -> 32.3 mm
- net /DTR: track 0.00 -> 23.5 mm, vias 0 -> 2
- net /M2_OUT2_N: track 0.00 -> 22.9 mm
- net /M2_OUT1_N: track 0.00 -> 22.6 mm
- net /M2_OUT2_P: track 0.00 -> 19.4 mm, vias 0 -> 2
- net /M2_OUT1_P: track 0.00 -> 18.8 mm, vias 0 -> 2
- net Net-(U10-V3P3OUT): track 0.00 -> 16.5 mm
- net /M1_OUT2_P: track 0.00 -> 15.8 mm, vias 0 -> 2
- net /M1_OUT2_N: track 0.00 -> 15.0 mm
- net /RTS: track 0.00 -> 14.6 mm
- net Net-(U3-V3P3OUT): track 0.00 -> 12.8 mm
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Other:
- board size 86.8 x 49 mm -> 83.1 x 45.4 mm

Commit message: 729
Parts:
- R5, R6: moved to F.Cu
- moved R6 12.9 mm to (86.2, 79.0), turned to 90 degrees
- moved R5 10.6 mm to (84.5, 79.1), turned to 90 degrees
- moved C20 4.32 mm to (49.4, 76.2), turned to -90 degrees
- moved C3 0.60 mm to (87.0, 87.1)
- moved C2 0.46 mm to (87.0, 88.8)
Connections:
- U15 pad 10: /M1_IN3 -> /DRV2_FAULT
- U15 pad 16: unconnected-(U15-IO13-Pad16) -> /M2_OUT2_CS
- U15 pad 22: unconnected-(U15-SDI/SD1-Pad22) -> /DRV1_FAULT
- U15 pad 24: unconnected-(U15-IO2-Pad24) -> /M1_IN3
- U15 pad 26: unconnected-(U15-IO4-Pad26) -> /M1_IN2
- U15 pad 27: /LED -> /M1_IN1
- U15 pad 28: /DRV1_FAULT -> unconnected-(U15-IO17-Pad28)
- U15 pad 30: /I2C1_SCL -> /I2C2_SCL
- U15 pad 31: /I2C1_SDA -> /I2C2_SDA
- U15 pad 33: /I2C2_SCL -> /I2C1_SCL
- U15 pad 36: /I2C2_SDA -> /I2C1_SDA
- U15 pad 37: /DRV2_FAULT -> unconnected-(U15-IO23-Pad37)
- U15 pad 6: /M2_OUT1_CS -> unconnected-(U15-IO34-Pad6)
- U15 pad 7: /M2_OUT2_CS -> unconnected-(U15-IO35-Pad7)
- U15 pad 8: /M1_IN1 -> /M2_OUT1_CS
- U15 pad 9: /M1_IN2 -> /LED
Routing:
- net /DRV1_EN: track 0.00 -> 38.7 mm, vias 0 -> 2
- net /M2_OUT1_CS: track 0.00 -> 36.4 mm, vias 0 -> 2
- net /M1_IN1: track 0.00 -> 34.2 mm, vias 0 -> 1
- net /M1_IN2: track 0.00 -> 33.7 mm, vias 0 -> 1
- net /DRV1_FAULT: track 2.73 -> 35.5 mm, vias 0 -> 2
- net /M1_IN3: track 0.00 -> 29.5 mm, vias 0 -> 2
- net Net-(U7-TXD): track 0.00 -> 24.8 mm, vias 0 -> 3
- net /M2_IN1: track 0.00 -> 23.7 mm, vias 0 -> 2
- net /M2_OUT2_CS: track 0.00 -> 23.3 mm, vias 0 -> 2
- net /DRV2_FAULT: track 2.90 -> 24.3 mm, vias 0 -> 3
- net /M2_IN2: track 0.00 -> 20.9 mm, vias 0 -> 2
- net Net-(U7-RXD): track 0.00 -> 20.4 mm, vias 0 -> 3
- net /DRV2_EN: track 0.00 -> 20.4 mm, vias 0 -> 3
- net +3V3: track 164.1 -> 183.2 mm, vias 6 -> 8
- net /M2_IN3: track 0.00 -> 17.0 mm, vias 0 -> 2
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Other:
- copper layers 2 -> 4
